Commit message: 1. added xacro file to simulate point cloud. but not working; 2. added explore_lite for autonomous exploration. to use, you need to install explore_lite package by ssudo apt-get install ros-kinetic-explore-lite, then run the cmd in launch/scribble.txt

File: urdf/turtlebot3_burger_jjiang_play.gazebo.xacro (robot description, xacro)
@@ -1,6 +1,6 @@
 <?xml version="1.0"?>
 <robot name="turtlebot3_burger_sim" xmlns:xacro="http://ros.org/wiki/xacro">
-  <xacro:arg name="laser_visual" default="true"/>
-  <xacro:arg name="imu_visual"   default="true"/>
+  <xacro:arg name="laser_visual" default="false"/>
+  <xacro:arg name="imu_visual"   default="false"/>
   <gazebo>
     <plugin name="turtlebot3_burger_controller" filename="libgazebo_ros_diff_drive.so">
@@ -120,4 +120,46 @@
     </sensor>
   </gazebo>
+  <!-- jjiang trys out point cloud -->
+  <gazebo reference="velodyne_base_link">
+    <material>Gazebo/DarkGrey</material>
+    <sensor type="ray" name="velodyne-VLP16">
+      <pose>0 0 0 0 0 0</pose>
+      <visualize>false</visualize>
+      <update_rate>10</update_rate>
+      <ray>
+        <scan>
+          <horizontal>
+            <samples>1875</samples>
+            <resolution>1</resolution>
+            <min_angle>0.0</min_angle>
+            <max_angle>6.28</max_angle>
+          </horizontal>
+          <vertical>
+            <samples>16</samples>
+            <resolution>1</resolution>
+            <min_angle>-0.261</min_angle>
+            <max_angle> 0.261</max_angle>
+          </vertical>
+        </scan>
+        <range>
+          <min>0.1</min>
+          <max>10</max>
+          <resolution>0.001</resolution>
+        </range>
+        <noise>
+          <type>gaussian</type>
+          <mean>0.0</mean>
+          <stddev>0.0</stddev>
+        </noise>
+      </ray>
+      <plugin name="gazebo_ros_laser_controller" filename="libgazebo_ros_velodyne_laser.so">
+        <topicName>/velodyne_points</topicName>
+        <frameName>velodyne</frameName>
+        <min_range>0.1</min_range>
+        <max_range>10</max_range>
+        <gaussianNoise>0.008</gaussianNoise>
+      </plugin>
+    </sensor>
+  </gazebo>
   <!-- camera -->
   <gazebo reference="base_camera">
